File: PEBBL3.brd (EAGLE design)
At the start: 106 x 49 mm, 30 parts, among them IC1 ESPWROOM32, J1 POWER_JACKPTH_SLOTS, U1 HY931147C-RJ45

Commit message: Experiments with dimensions
Parts:
- removed J1: POWER_JACKPTH_SLOTS, freetronics-jon:POWER_JACK_PTH_SLOTS
- removed JP1, JP4: M06X2, freetronics-jon:2X6-SHROUDED
- removed JP3: (no value), freetronics-jon:1X04
- removed REG1: AG9900, freetronics-jon:AG9900
- removed REG2: K7805-500R3, freetronics-jon:K78XX-500R3
- removed RN5: 49R9 1%, freetronics-master-v1:CAY16
- removed S2: FLASH, freetronics-jon:TACTILE_SWITCH_SMD_2PIN_TINY
- added C5: 0.1uF, SparkFun-Capacitors:0603-CAP
- added IC2: LTC4054, freetronics-luke:SOT23-5
- added LED1: ORANGE, freetronics-master-v1:LED-0603
- added R9: 10K, SparkFun-Resistors:0603-RES
- added S3, S4, S5, S6: MOMENTARY-SWITCH-SPST-SMD-5.2MM, SparkFun-Switches:TACTILE_SWITCH_SMD_5.2MM
- added S7: 2P-JST-PTH, freetronics-jon:JST-2MM-TH-RA
- added U$3: CP2104, freetronics-jon:QFN-24
- added U$6: M06X2RA, freetronics-jon:2X6-SHROUDED-RA
- C2: value (none) -> 1uF 0603; device freetronics-jon:0805 -> freetronics:0603
- C4: value 100uF 25V -> 0.1uF; device rcl:PANASONIC_D -> SparkFun-Capacitors:0603-CAP
- R1, R2: device freetronics:0603@2 -> freetronics:0603
- R3: value 10K -> 1K 0603; device freetronics:0603@2 -> freetronics:0603
- R4: value 10K -> 10K 0603; device freetronics:0603@2 -> freetronics:0603
- R6: value 10K -> 4K7; device freetronics:0603@2 -> freetronics:0603
- R7, R8: device freetronics:0603@2 -> SparkFun-Resistors:0603-RES
- S1: device freetronics-jon:TACTILE_SWITCH_SMD_2PIN_TINY -> freetronics-jon:TACT-VERT-1TAB
- U$1: value LAN8720 -> USB-C; device microchip-smsc-lan8720:QFN24 -> freetronics-jon:USB-C-U52A
- U$2: value FEATHER -> AP2112KSOT25; device freetronics-jon:FEATHER -> freetronics-jon:SOT23-5
- U1: value HY931147C-RJ45 -> MPU-9250; device freetronics-jon:HY931147C -> Testing:QFN24_PAD
- moved JP2 66.1 mm to (5.00, 28.0)
- moved FID2 65.1 mm to (48.5, 42.0)
- moved FID3 60.3 mm to (50.0, 35.0)
- moved FID1 51.0 mm to (59.0, 30.0)
- moved S1 50.6 mm to (7.00, 40.6), flipped to the bottom, turned to 180 degrees
- moved U$2 39.8 mm to (12.0, 32.0), turned to 0 degrees
- moved C4 38.0 mm to (-11.0, 27.0), turned to 0 degrees
- moved R8 36.9 mm to (-11.0, 30.0)
- moved R7 31.9 mm to (-7.00, 30.0)
- moved R2 30.1 mm to (34.0, 27.0), turned to 90 degrees
- moved IC1 28.4 mm to (34.5, 24.0), flipped to the bottom, turned to 90 degrees
- moved LED10 24.3 mm to (12.0, 39.0)
- moved R5 21.0 mm to (12.0, 42.0), turned to 180 degrees
- moved U1 20.1 mm to (-11.0, 40.0)
- moved R1 16.2 mm to (32.0, 9.00), turned to 180 degrees
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Connections:
- removed net BUTTON1: JP4.1
- removed net BUTTON2: JP4.2
- removed net BUTTON3: JP4.3
- removed net BUTTON4: JP4.4
- removed net N$1: RN5.1, U$1.21, U1.P$5
- removed net N$11: R3.2, U$1.11
- removed net N$12: C2.1, R7.2, U$1.15
- removed net N$13: R8.2, U$1.12
- removed net N$5: RN5.3, RN5.4, U$1.23, U1.P$1
- removed net N$7: U$1.1, U$1.19
- removed net N$9: R6.2, U$1.8
- removed net VDDCR: U$1.6
- new net !CS: R9.1, U1.22
- new net FSYNC: U1.11
- new net GND_PAD: U$3.TGND
- new net INT: U1.12
- new net REGIN: U$3.7
- new net REGOUT: C4.1, U1.10
- new net SCL/SCLK: R8.1, U1.23
- new net SDA/SDI: R7.1, U1.24
- new net V+: U$1.A4, U$1.A9, U$1.B4, U$1.B9
- new net VDD: C5.1, U$3.6, U1.13
- net 3.3V: now also U$2.5, U$6.11; no longer JP1.11, JP3.1, JP4.11, R3.1, R4.1, R6.1, R7.1, R8.1, REG2.3
- net BUTTON5: no longer JP4.5
- net BUTTON6: no longer JP4.6
- net BUTTON7: no longer JP4.7
- net BUTTON8: no longer JP4.8
- net DATA1: now also U$6.1; no longer JP1.1
- net DATA2: now also U$6.2; no longer JP1.2
- net DATA3: now also U$6.3; no longer JP1.3
- net DATA4: now also U$6.4; no longer JP1.4
- net DATA5: now also U$6.5; no longer JP1.5
- net DATA6: now also U$6.6; no longer JP1.6
- net DATA7: now also U$6.7; no longer JP1.7
- net DATA8: now also U$6.8; no longer JP1.8
- net EN: now also U$6.12; no longer JP1.12, JP4.12
- net GND: now also C2.1, C4.2, C5.2, IC2.2, R6.2, S7.NEG, U$1.A1, U$1.A12, U$1.B1, U$1.B12, U$1.CASE1, U$1.CASE2, U$1.CASE3, U$1.CASE4, U$1.FIX1, U$1.FIX2, U$1.FIX3, U$1.FIX4, U$2.2, U$3.2, U$6.10, U1.18, U1.20, U1.9, U1.CENTER; no longer C2.2, C4.-, J1.GND, J1.GNDBREAK, JP1.10, JP3.4, JP4.10, REG1.P3, REG2.2, RN5.5, RN5.6, RN5.7, RN5.8, S2.2, U$1.EXP, U1.GND1, U1.GND2
- net GPIO0: no longer S2.1
- net N$2: now also C2.2, IC2.4, R3.1, R4.1; no longer REG1.P5, REG1.P6, U1.P$9
- net N$3: now also IC2.5, R6.1; no longer REG1.P7, REG1.P8, U1.P$10
- net N$4: now also IC2.3, S7.POS; no longer RN5.2, U$1.20, U1.P$6
- net N$6: now also IC2.1, LED1.C, R4.2; no longer U$1.22, U1.P$2
- net N$8: now also LED1.A, R3.2; no longer R4.2, U$1.7
- net RXD0: no longer JP3.2
- net TXD0: no longer JP3.3
- net VCC: now also U$2.1, U$6.9; no longer C4.+, J1.PWR, JP1.9, JP4.9, REG1.P1, REG1.P2, REG2.1
- net VDDIO: now also R7.2, R8.2, R9.2, U1.1, U1.8; no longer U$1.9
Routing:
- net 3.3V: track 14.3 -> 0.00 mm
- net GPIO0: track 12.5 -> 0.00 mm, vias 1 -> 0
- net DATA5: track 6.22 -> 0.00 mm
- net BUTTON6: track 6.03 -> 0.00 mm
- net BUTTON8: track 5.63 -> 0.00 mm, vias 1 -> 0
- net DATA6: track 3.31 -> 0.00 mm
- net BUTTON7: track 3.21 -> 0.00 mm
- net IO33: track 2.84 -> 0.00 mm
Other:
- board size 106 x 49 mm -> 44 x 44 mm
- board text added: "PEBBL3"
- board text added: "www.superhouse.tv/pebbl3"
- board text removed: "3"
- board text removed: "ESP32 LAN / POE"
- board text removed: "FLASH"
- board text removed: "G"
- board text removed: "R"
- board text removed: "T"
- board text removed: "www.superhouse.tv"
