File: PEBBL3.sch (EAGLE design)
At the start: 30 parts, among them IC1 ESPWROOM32, J1 POWER_JACKPTH_SLOTS, U1 HY931147C-RJ45

Commit message: Experiments with dimensions
Parts:
- removed J1: POWER_JACKPTH_SLOTS, freetronics-jon:POWER_JACKPTH_SLOTS
- removed JP1, JP4: M06X2, freetronics-jon:M06X2
- removed JP3: (no value), freetronics-jon:M04PTH
- removed REG1: AG9900, freetronics-jon:AG9900
- removed REG2: K7805-500R3, freetronics-jon:K78XX-500R3
- removed RN5: 49R9 1%, freetronics-master-v1:4R-NCAY16
- removed S2: FLASH, freetronics-jon:TAC_SWITCH_2PINSMT
- added C5: 0.1uF, SparkFun-Capacitors:0.1UF-25V(+80/-20%)(0603)
- added IC2: LTC4054, freetronics-luke:LTC4054
- added LED1: ORANGE, freetronics-master-v1:LED0603
- added R9: 10K, SparkFun-Resistors:10KOHM-1/10W-1%(0603)0603
- added S3, S4, S5, S6: MOMENTARY-SWITCH-SPST-SMD-5.2MM, SparkFun-Switches:MOMENTARY-SWITCH-SPST-SMD-5.2MM
- added S7: 2P-JST-PTH, freetronics-jon:2P-JST-TH-RAPTH
- added U$3: CP2104, freetronics-jon:CP2104
- added U$6: M06X2RA, freetronics-jon:M06X2RA
- C2: value (none) -> 1uF 0603; device freetronics-jon:CAP0805 -> freetronics:CAP0603
- C4: value 100uF 25V -> 0.1uF; device rcl:CPOL-EUD -> SparkFun-Capacitors:0.1UF-25V(+80/-20%)(0603)
- R3: value 10K -> 1K 0603
- R4: value 10K -> 10K 0603
- R6: value 10K -> 4K7
- R7, R8: device freetronics:RESISTOR0603 -> SparkFun-Resistors:10KOHM-1/10W-1%(0603)0603
- S1: device freetronics-jon:TAC_SWITCH_2PINSMT -> freetronics-jon:TAC-SWITCH-1TAB
- U$1: value LAN8720 -> USB-C; device microchip-smsc-lan8720:LAN8720 -> freetronics-jon:USB-C
- U$2: value FEATHER -> AP2112KSOT25; device freetronics-jon:FEATHER -> freetronics-jon:AP2112KSOT25
- U1: value HY931147C-RJ45 -> MPU-9250; device freetronics-jon:HY931147C-RJ45 -> Testing:MPU-9250
Connections:
- removed net BUTTON1: JP4.1
- removed net BUTTON2: JP4.2
- removed net BUTTON3: JP4.3
- removed net BUTTON4: JP4.4
- removed net N$1: RN5A.1, U$1.TXP, U1.TX+
- removed net N$11: R3.2, U$1.CRS_DV/MODE2
- removed net N$12: C2.1, R7.2, U$1.!RST
- removed net N$13: R8.2, U$1.MDIO
- removed net N$5: RN5C.1, RN5D.1, U$1.RXP, U1.RX+
- removed net N$7: U$1.VDD1A, U$1.VDD2A
- removed net N$9: R6.2, U$1.RXD0/MODE0
- new net !CS: R9.1, U1.!CS
- new net FSYNC: U1.FSYNC
- new net INT: U1.INT
- new net REGOUT: C4.1, U1.REGOUT
- new net SCL/SCLK: R8.1, U1.SCL/SCLK
- new net SDA/SDI: R7.1, U1.SDA/SDI
- new net VDD: C5.1, U1.VDD
- new net VDDIO: R7.2, R8.2, R9.2, U1.VDDIO
- net 3.3V: now also U$2.VOUT, U$6.11; no longer JP1.11, JP3.1, JP4.11, R3.1, R4.1, R6.1, R7.1, R8.1, REG2.OUT
- net BUTTON5: no longer JP4.5
- net BUTTON6: no longer JP4.6
- net BUTTON7: no longer JP4.7
- net BUTTON8: no longer JP4.8
- net DATA1: now also U$6.1; no longer JP1.1
- net DATA2: now also U$6.2; no longer JP1.2
- net DATA3: now also U$6.3; no longer JP1.3
- net DATA4: now also U$6.4; no longer JP1.4
- net DATA5: now also U$6.5; no longer JP1.5
- net DATA6: now also U$6.6; no longer JP1.6
- net DATA7: now also U$6.7; no longer JP1.7
- net DATA8: now also U$6.8; no longer JP1.8
- net EN: now also S1.2, U$6.12; no longer JP1.12, JP4.12, S1.S
- net GND: now also C2.1, C4.2, C5.2, IC2.GND, R6.2, S1.1, S7.NEG, U$2.GND, U$6.10, U1.AD0/SDO, U1.GND; no longer C2.2, C4.-, J1.GND, J1.GNDBREAK, JP1.10, JP3.4, JP4.10, REG1.-VDC, REG2.GND, RN5A.2, RN5B.2, RN5C.2, RN5D.2, S1.P, S2.S, U$1.VSS, U1.GND1, U1.GND2
- net GPIO0: no longer S2.P
- net N$2: now also C2.2, IC2.VCC, R3.1, R4.1; no longer REG1.VIN+1, REG1.VIN+2, U1.V+
- net N$3: now also IC2.PROG, R6.1; no longer REG1.VIN-1, REG1.VIN-2, U1.V-
- net N$4: now also IC2.BAT, S7.POS; no longer RN5B.1, U$1.TXN, U1.TX-
- net N$6: now also IC2.!CHRG, LED1.C, R4.2; no longer U$1.RXN, U1.RX-
- net N$8: now also LED1.A, R3.2; no longer R4.2, U$1.RXD1/MODE1
- net RXD0: no longer JP3.2
- net TXD0: no longer JP3.3
- net VCC: now also U$2.VIN, U$6.9; no longer C4.+, J1.PWR, JP1.9, JP4.9, REG1.+VDC1, REG1.+VDC2, REG2.IN
Other:
- note added: "2.0mm JST"
- note added: "AD0/SDO defaults to 0V. This sets the I2C address to 0b1101000 (0x68)"
- note added: "Charge"
- note added: "ESP32 Module with I/O Breakout"
- note added: "Output"
- note added: "R6=4K7 gives 200mA charge rate (1C 200mA/h)"
- note added: "SKU: PEBBL3"
- note added: "TODO: Add battery power switch Add IMU Add battery charge sensor Change reset button to right angle Connect CHRG output to GPIO Add auto reset transistors Link TX/RX to cp2101n Replace CP2102 with CP2102N? Battery options: - https://www.banggood.com/5PCS-3_7V-300mAh-25C-Lipo-Battery-Charger-Set-for-H8-H22-Eachine-H8-mini-RC-Quadcopter-p-1380233.html - https://hobbyking.com/en_us/turnigy-2000mah-1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"
- note added: "V1.0 (2019-01-26)"
- note added: "www.superhouse.tv/pebbl3"
- note removed: "ACTIVITY"
- note removed: "ESP32 Module with LAN & PoE"
- note removed: "LINK"
- note removed: "SKU: POESP32"
- note removed: "V1.0 (2018-06-15)"
- note removed: "www.superhouse.tv/poesp32"
- moved on the sheet: C2, JP2, R3, R4, R6
